File: KnaveOfWorry.sch (KiCad schematic (older format))
At the start: 60 parts, among them U1 PIC18F27Q43-PDIP28

Commit message: some progress, gonna check old thing
Parts:
- removed D?: 1N4001, Diode_THT:D_DO-41_SOD81_P7.62mm_Horizontal, symbol Device:D
- added C7: 10uf, Capacitor_THT:CP_Radial_D5.0mm_P2.00mm, symbol Device:CP
- added SW2: SW_Push, Button_Switch_THT:SW_PUSH_6mm, symbol Switch:SW_Push
- added SW3: SW_SPDT, HammerheadAudio:Tayda_Slide_SPDT, symbol Switch:SW_SPDT
- added U4: 5V Regulator, HammerheadAudio:BR300, symbol Regulator_Linear:L7805
- C1, C3: renamed from C?; footprint (none) -> Capacitor_THT:C_Disc_D3.0mm_W2.0mm_P2.50mm
- C6: renamed from C?; footprint Capacitor_THT:CP_Radial_D5.0mm_P2.00mm -> Capacitor_THT:CP_Radial_D8.0mm_P2.50mm
- D1, D2, D3, D4, D5, D6, D7, D8, D9: footprint (none) -> LED_THT:LED_D3.0mm
- D10, D11, D12, D13, D14, D15, D16: footprint (none) -> LED_THT:LED_D5.0mm
- D18, D20: renamed from D?; footprint (none) -> LED_THT:LED_D5.0mm
- D21: renamed from D?; footprint (none) -> HammerheadAudio:DO-35-P5mm
- J1: renamed from J?; footprint (none) -> Connector_PinHeader_2.54mm:PinHeader_1x06_P2.54mm_Vertical
- LS1: renamed from LS?; footprint (none) -> HammerheadAudio:Speaker-DBU-SM420608-1
- R1, R10, R11, R12, R13, R2, R3, R5, R6, R7, R8, R9: renamed from R?; footprint (none) -> HammerheadAudio:R_THT_P7.62
- RV1, RV2: renamed from RV?; footprint (none) -> HammerheadAudio:PT-6-V_FixedPads
- U1: footprint (none) -> Package_DIP:DIP-28_W7.62mm_Socket
- U2, U3: renamed from U?; footprint (none) -> Package_DIP:DIP-8_W7.62mm_Socket
- gave numbers to parts that had none: 16
Connections:
- net +5V: now also C7.1, SW2.1, U4.3 (OUT)
- net GND: now also C7.2, U4.2 (GND)
- net PIC_DECLINE: now also SW2.2
- net VCC: now also U4.1 (IN)
- net at LS1.1: now also SW3.1 (A); no longer C6.2
- new net: C6.2, SW3.2 (B)
- no-connect marks 6 -> 7
Other:
- moved on the sheet: J9, LS1, R12, R13

Commit message: commit before plaing 3mm LEDs
Parts:
- D1, D2, D3, D4, D5, D6, D7, D8, D9: footprint LED_THT:LED_D3.0mm -> HammerheadAudio:LED_D3.0mm_Centered_NoRef
- D10, D11, D12, D13, D14, D15, D16: footprint LED_THT:LED_D5.0mm -> HammerheadAudio:LED_Centered_NoRef
Changed lines of the file:
@@
 F 0 "D1" H 3443 2045 50  0000 C CNN
 F 1 "LED_ALT" H 3443 2136 50  0000 C CNN
-F 2 "LED_THT:LED_D3.0mm" H 3450 2300 50  0001 C CNN
+F 2 "HammerheadAudio:LED_D3.0mm_Centered_NoRef" H 3450 2300 50  0001 C CNN
 F 3 "~" H 3450 2300 50  0001 C CNN
 	1    3450 2300
@@
 F 0 "D2" H 3743 2295 50  0000 C CNN
 F 1 "LED_ALT" H 3743 2386 50  0000 C CNN
-F 2 "LED_THT:LED_D3.0mm" H 3750 2550 50  0001 C CNN
+F 2 "HammerheadAudio:LED_D3.0mm_Centered_NoRef" H 3750 2550 50  0001 C CNN
 F 3 "~" H 3750 2550 50  0001 C CNN
 	1    3750 2550
@@
 F 0 "D3" H 3443 2545 50  0000 C CNN
 F 1 "LED_ALT" H 3443 2636 50  0000 C CNN
-F 2 "LED_THT:LED_D3.0mm" H 3450 2800 50  0001 C CNN
+F 2 "HammerheadAudio:LED_D3.0mm_Centered_NoRef" H 3450 2800 50  0001 C CNN
 F 3 "~" H 3450 2800 50  0001 C CNN
 	1    3450 2800
@@
 F 0 "D4" H 3743 2795 50  0000 C CNN
 F 1 "LED_ALT" H 3743 2886 50  0000 C CNN
-F 2 "LED_THT:LED_D3.0mm" H 3750 3050 50  0001 C CNN
+F 2 "HammerheadAudio:LED_D3.0mm_Centered_NoRef" H 3750 3050 50  0001 C CNN
 F 3 "~" H 3750 3050 50  0001 C CNN
 	1    3750 3050
@@
 F 0 "D5" H 3443 3045 50  0000 C CNN
 F 1 "LED_ALT" H 3443 3136 50  0000 C CNN
-F 2 "LED_THT:LED_D3.0mm" H 3450 3300 50  0001 C CNN
+F 2 "HammerheadAudio:LED_D3.0mm_Centered_NoRef" H 3450 3300 50  0001 C CNN
 F 3 "~" H 3450 3300 50  0001 C CNN
 	1    3450 3300
@@
 F 0 "D6" H 3443 3795 50  0000 C CNN
 F 1 "LED_ALT" H 3443 3886 50  0000 C CNN
-F 2 "LED_THT:LED_D3.0mm" H 3450 4050 50  0001 C CNN
+F 2 "HammerheadAudio:LED_D3.0mm_Centered_NoRef" H 3450 4050 50  0001 C CNN
 F 3 "~" H 3450 4050 50  0001 C CNN
 	1    3450 4050
@@
 F 0 "D7" H 3743 4045 50  0000 C CNN
 F 1 "LED_ALT" H 3743 4136 50  0000 C CNN
-F 2 "LED_THT:LED_D3.0mm" H 3750 4300 50  0001 C CNN
+F 2 "HammerheadAudio:LED_D3.0mm_Centered_NoRef" H 3750 4300 50  0001 C CNN
 F 3 "~" H 3750 4300 50  0001 C CNN
 	1    3750 4300
@@
 F 0 "D8" H 3443 4295 50  0000 C CNN
 F 1 "LED_ALT" H 3443 4386 50  0000 C CNN
-F 2 "LED_THT:LED_D3.0mm" H 3450 4550 50  0001 C CNN
+F 2 "HammerheadAudio:LED_D3.0mm_Centered_NoRef" H 3450 4550 50  0001 C CNN
 F 3 "~" H 3450 4550 50  0001 C CNN
 	1    3450 4550
@@
 F 0 "D9" H 3743 4545 50  0000 C CNN
 F 1 "LED_ALT" H 3743 4636 50  0000 C CNN
-F 2 "LED_THT:LED_D3.0mm" H 3750 4800 50  0001 C CNN
+F 2 "HammerheadAudio:LED_D3.0mm_Centered_NoRef" H 3750 4800 50  0001 C CNN
 F 3 "~" H 3750 4800 50  0001 C CNN
 	1    3750 4800
@@
 F 0 "D16" H 1593 5016 50  0000 C CNN
 F 1 "LED" H 1593 4925 50  0000 C CNN
-F 2 "LED_THT:LED_D5.0mm" H 1600 4800 50  0001 C CNN
+F 2 "HammerheadAudio:LED_Centered_NoRef" H 1600 4800 50  0001 C CNN
 F 3 "~" H 1600 4800 50  0001 C CNN
 	1    1600 4800
@@
 F 0 "D15" H 1343 4766 50  0000 C CNN
 F 1 "LED" H 1343 4675 50  0000 C CNN
-F 2 "LED_THT:LED_D5.0mm" H 1350 4550 50  0001 C CNN
+F 2 "HammerheadAudio:LED_Centered_NoRef" H 1350 4550 50  0001 C CNN
 F 3 "~" H 1350 4550 50  0001 C CNN
 	1    1350 4550
@@
 F 0 "D14" H 1593 4516 50  0000 C CNN
 F 1 "LED" H 1593 4425 50  0000 C CNN
-F 2 "LED_THT:LED_D5.0mm" H 1600 4300 50  0001 C CNN
+F 2 "HammerheadAudio:LED_Centered_NoRef" H 1600 4300 50  0001 C CNN
 F 3 "~" H 1600 4300 50  0001 C CNN
 	1    1600 4300
@@
 F 0 "D13" H 1343 4266 50  0000 C CNN
 F 1 "LED" H 1343 4175 50  0000 C CNN
-F 2 "LED_THT:LED_D5.0mm" H 1350 4050 50  0001 C CNN
+F 2 "HammerheadAudio:LED_Centered_NoRef" H 1350 4050 50  0001 C CNN
 F 3 "~" H 1350 4050 50  0001 C CNN
 	1    1350 4050
@@
 F 0 "D12" H 1593 4016 50  0000 C CNN
 F 1 "LED" H 1593 3925 50  0000 C CNN
-F 2 "LED_THT:LED_D5.0mm" H 1600 3800 50  0001 C CNN
+F 2 "HammerheadAudio:LED_Centered_NoRef" H 1600 3800 50  0001 C CNN
 F 3 "~" H 1600 3800 50  0001 C CNN
 	1    1600 3800
@@
 F 0 "D11" H 1343 3766 50  0000 C CNN
 F 1 "LED" H 1343 3675 50  0000 C CNN
-F 2 "LED_THT:LED_D5.0mm" H 1350 3550 50  0001 C CNN
+F 2 "HammerheadAudio:LED_Centered_NoRef" H 1350 3550 50  0001 C CNN
 F 3 "~" H 1350 3550 50  0001 C CNN
 	1    1350 3550
@@
 F 0 "D10" H 1593 3266 50  0000 C CNN
 F 1 "LED" H 1593 3175 50  0000 C CNN
-F 2 "LED_THT:LED_D5.0mm" H 1600 3050 50  0001 C CNN
+F 2 "HammerheadAudio:LED_Centered_NoRef" H 1600 3050 50  0001 C CNN
 F 3 "~" H 1600 3050 50  0001 C CNN
 	1    1600 3050
