File: KnaveOfWorry.sch (KiCad schematic (older format))
At the start: 61 parts, among them J1 Conn_01x06_Female, J2 Eurojack, J3 PWR_IN_PHNX, J4 PWR_IN_PHNX, J5 PWR_IN_PHNX, J6 PWR_IN_PHNX, J7 CLK_IN, J8 MCLR_IN, J9 DECLINE_IN, Q1 2N3904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

Commit message: commit before laying down traces
Parts:
- removed R5: 100k, HammerheadAudio:R_THT_P7.62, symbol Device:R
- renumbered R13 to R5
Connections:
- net OUT_BUILTIN: now also U3.3 (+); no longer RV2.3
- net at J2.1 (Pin_1): now also RV2.2; no longer C2.2
- new net: C2.2, RV2.3
Other:
- moved on the sheet: J2, RV2
Changed lines of the file:
@@
 $EndComp
 $Comp
-L Device:R R13
+L Device:R R5
 U 1 1 5ED27BF6
 P 6150 6400
-F 0 "R13" H 6080 6354 50  0000 R CNN
+F 0 "R5" H 6080 6354 50  0000 R CNN
 F 1 "1M" H 6080 6445 50  0000 R CNN
 F 2 "HammerheadAudio:R_THT_P7.62" V 6080 6400 50  0001 C CNN
@@
 Wire Wire Line
 	7450 1100 7500 1100
-$Comp
-L Device:R R5
-U 1 1 5EDDAB43
-P 7850 1300
-F 0 "R5" H 7780 1254 50  0000 R CNN
-F 1 "100k" H 7780 1345 50  0000 R CNN
-F 2 "HammerheadAudio:R_THT_P7.62" V 7780 1300 50  0001 C CNN
-F 3 "~" H 7850 1300 50  0001 C CNN
-	1    7850 1300
-	-1   0    0    1
-$EndComp
-$Comp
-L Connector:Conn_01x03_Female J2
-U 1 1 5E236837
-P 8500 1500
-F 0 "J2" H 8528 1526 50  0000 L CNN
-F 1 "Eurojack" H 8528 1435 50  0000 L CNN
-F 2 "HammerheadAudio:EuroJack_MonoSW_THT" H 8500 1500 50  0001 C CNN
-F 3 "~" H 8500 1500 50  0001 C CNN
-	1    8500 1500
-	1    0    0    -1
-$EndComp
-Text GLabel 8200 1600 0    50   Input ~ 0
+Text GLabel 8150 1550 3    50   Input ~ 0
 OUT_BUILTIN
-$Comp
-L power:GND #PWR012
-U 1 1 5E237198
-P 7550 1500
-F 0 "#PWR012" H 7550 1250 50  0001 C CNN
-F 1 "GND" H 7555 1327 50  0000 C CNN
-F 2 "" H 7550 1500 50  0001 C CNN
-F 3 "" H 7550 1500 50  0001 C CNN
-	1    7550 1500
-	1    0    0    -1
-$EndComp
-Wire Wire Line
-	8200 1600 8300 1600
-Wire Wire Line
-	7550 1500 7850 1500
-Wire Wire Line
-	8200 1400 8300 1400
-Wire Wire Line
-	7800 1100 7850 1100
-Wire Wire Line
-	7850 1100 7850 1150
-Wire Wire Line
-	7850 1450 7850 1500
-Connection ~ 7850 1500
-Wire Wire Line
-	7850 1500 8300 1500
-Wire Wire Line
-	7850 1100 8200 1100
-Wire Wire Line
-	8200 1100 8200 1400
-Connection ~ 7850 1100
+Wire Wire Line
+	8150 1550 8250 1550
 $Comp
 L Amplifier_Audio:LM386 U3
@@
 L Device:R_POT_TRIM RV2
 U 1 1 5EEEB604
-P 5300 2650
-F 0 "RV2" H 5230 2604 50  0000 R CNN
-F 1 "R_POT_TRIM" H 5230 2695 50  0000 R CNN
-F 2 "HammerheadAudio:PT-6-V_FixedPads" H 5300 2650 50  0001 C CNN
-F 3 "~" H 5300 2650 50  0001 C CNN
-	1    5300 2650
+P 7850 1350
+F 0 "RV2" H 7780 1304 50  0000 R CNN
+F 1 "R_POT_TRIM" H 7780 1395 50  0000 R CNN
+F 2 "HammerheadAudio:PT-6-V_FixedPads" H 7850 1350 50  0001 C CNN
+F 3 "~" H 7850 1350 50  0001 C CNN
+	1    7850 1350
 	1    0    0    1
 $EndComp
@@
 L power:GND #PWR019
 U 1 1 5EEEB60E
-P 5300 2850
-F 0 "#PWR019" H 5300 2600 50  0001 C CNN
-F 1 "GND" H 5305 2677 50  0000 C CNN
-F 2 "" H 5300 2850 50  0001 C CNN
-F 3 "" H 5300 2850 50  0001 C CNN
-	1    5300 2850
-	1    0    0    -1
-$EndComp
-Wire Wire Line
-	5300 2500 5300 2450
-Wire Wire Line
-	5300 2850 5300 2800
+P 7850 1550
+F 0 "#PWR019" H 7850 1300 50  0001 C CNN
+F 1 "GND" H 7855 1377 50  0000 C CNN
+F 2 "" H 7850 1550 50  0001 C CNN
+F 3 "" H 7850 1550 50  0001 C CNN
+	1    7850 1550
+	1    0    0    -1
+$EndComp
+Wire Wire Line
+	7850 1550 7850 1500
 $Comp
 L power:GND #PWR020
@@
 Wire Wire Line
 	6250 2400 6250 2450
-Text GLabel 5300 2450 1    50   Input ~ 0
+Text GLabel 5450 2650 0    50   Input ~ 0
 OUT_BUILTIN
 $Comp
@@
 Wire Wire Line
 	9400 2800 9800 2800
+Wire Wire Line
+	7800 1100 7850 1100
+Wire Wire Line
+	7850 1100 7850 1200
+$Comp
+L Connector:Conn_01x03_Female J2
+U 1 1 5E236837
+P 8450 1450
+F 0 "J2" H 8478 1476 50  0000 L CNN
+F 1 "Eurojack" H 8478 1385 50  0000 L CNN
+F 2 "HammerheadAudio:EuroJack_MonoSW_THT" H 8450 1450 50  0001 C CNN
+F 3 "~" H 8450 1450 50  0001 C CNN
+	1    8450 1450
+	1    0    0    -1
+$EndComp
+Wire Wire Line
+	8000 1350 8250 1350
+$Comp
+L power:GND #PWR0102
+U 1 1 5EBD81BD
+P 8200 1450
+F 0 "#PWR0102" H 8200 1200 50  0001 C CNN
+F 1 "GND" H 8205 1277 50  0000 C CNN
+F 2 "" H 8200 1450 50  0001 C CNN
+F 3 "" H 8200 1450 50  0001 C CNN
+	1    8200 1450
+	0    1    1    0
+$EndComp
+Wire Wire Line
+	8200 1450 8250 1450
 $EndSCHEMATC

Commit message: commit before laying down traces
Parts:
- added LS2: Speaker, HammerheadAudio:Speaker-DBU-SM420608-1, symbol Device:Speaker
Connections:
- net GND: now also LS2.1
- net at U1.10 (RA6): now also D14.2 (A); no longer D12.2 (A)
- net at U1.12 (RC1): now also D12.2 (A); no longer D14.2 (A)
- net at U1.13 (RC2): now also D11.2 (A); no longer D15.2 (A)
- net at U1.14 (RC3): now also D10.2 (A); no longer D16.2 (A)
- net at U1.15 (RC4): now also D1.2 (A); no longer D9.2 (A)
- net at U1.16 (RC5): now also D2.2 (A); no longer D8.2 (A)
- net at U1.17 (RC6): now also D3.2 (A); no longer D7.2 (A)
- net at U1.18 (RC7): now also D4.2 (A); no longer D6.2 (A)
- net at U1.22 (RB1): now also D6.2 (A); no longer D4.2 (A)
- net at U1.23 (RB2): now also D7.2 (A); no longer D3.2 (A)
- net at U1.24 (RB3): now also D8.2 (A); no longer D2.2 (A)
- net at U1.25 (RB4): now also D9.2 (A); no longer D1.2 (A)
- net at U1.7 (RA5): now also D16.2 (A); no longer D10.2 (A)
- net at U1.9 (RA7): now also D15.2 (A); no longer D11.2 (A)
- net at LS1.1, SW3.1 (A): now also LS2.2
Other:
- moved on the sheet: D1, D10, D11, D12, D13, D14, D15, D16, D2, D3, D4, D5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
